File: circuit-design/Circuito de potencia genérico.kicad_pcb (KiCad board)
At the start: 2 copper layers, 7 parts, among them J1 Screw_Terminal_1x04, J2 CONN_01X06

Commit message: Archivos kicad de placa power
Parts:
- ACS712-20A1, ACS712-20A2, J1, J2, PowerSupply_5V1, Relay1, Relay2: moved to F.Cu
- moved PowerSupply_5V1 133.1 mm to (104.1, 44.5), turned to 0 degrees
- moved J2 115.3 mm to (118.1, 82.5)
- moved ACS712-20A1 90.9 mm to (127.0, 50.8), turned to 0 degrees
- moved ACS712-20A2 90.9 mm to (127.0, 64.8), turned to 0 degrees
- moved J1 76.1 mm to (134.6, 45.7), turned to 0 degrees
- moved Relay1 32.5 mm to (158.8, 40.6), turned to 0 degrees
- moved Relay2 24.0 mm to (177.8, 40.6), turned to 0 degrees
Routing:
- net Net-(ACS712-20A2-Pad5): track 61.1 -> 290.8 mm
- net Net-(J1-Pad2): track 88.5 -> 209.2 mm
- net Net-(ACS712-20A2-Pad4): track 31.0 -> 135.1 mm
- net Net-(ACS712-20A1-Pad5): track 20.8 -> 60.9 mm
- net Net-(J1-Pad1): track 18.8 -> 51.4 mm
- net Net-(ACS712-20A1-Pad4): track 12.0 -> 29.5 mm
- net Net-(ACS712-20A1-Pad3): track 150.3 -> 159.8 mm
- net Net-(ACS712-20A1-Pad1): track 213.6 -> 204.5 mm
- net Net-(J2-Pad6): track 50.6 -> 43.7 mm
- net Net-(J2-Pad5): track 74.7 -> 68.1 mm
- net Net-(ACS712-20A1-Pad2): track 33.3 -> 31.0 mm
- net Net-(ACS712-20A2-Pad2): track 21.9 -> 20.6 mm
Other:
- net class 220V added: clearance 0.2, trace_width 3, via_dia 3, via_drill 1.2
- net class 220V angosto added: clearance 0.2, trace_width 3, via_dia 3, via_drill 1
- net class 5V added: clearance 0.2, trace_width 2, via_dia 1.2, via_drill 1
- net class Default: trace_width 1 -> 1.3; via_dia 1 -> 1.3; via_drill 0.4 -> 1.2
- rule pad_to_mask_clearance: 0.2 -> 0
- rule trace_min: 0.3 -> 0.2
- board text removed: "DqR PowerBoard v1.0"
