File: circuit-design/Circuito de potencia genérico.sch (KiCad schematic (older format))
At the start: 7 parts, among them J1 Screw_Terminal_1x04, J2 CONN_01X06

Commit message: Archivos kicad de placa power
Parts:
- PowerSupply_5V1: symbol PowerSupply_5V-RESCUE-Circuito_de_potencia_genérico -> PowerSupply_5V
Connections:
- wire segments 51 -> 52
Other:
- moved on the sheet: J1, J2
Changed lines of the file:
@@
 L ACS712-20A ACS712-20A2
 U 1 1 5986365D
-P 5550 2700
-F 0 "ACS712-20A2" V 5550 2700 60  0001 R TNN
-F 1 "ACS712-20A" H 5550 2700 60  0001 R TNN
-F 2 "Huellas de Componentes DqR:ACS712" H 5550 2700 60  0001 C CNN
-F 3 "" H 5550 2700 60  0001 C CNN
-	1    5550 2700
+P 5200 3300
+F 0 "ACS712-20A2" V 5200 3300 60  0001 R TNN
+F 1 "ACS712-20A" H 5200 3300 60  0001 R TNN
+F 2 "Huellas de Componentes DqR:ACS712" H 5200 3300 60  0001 C CNN
+F 3 "" H 5200 3300 60  0001 C CNN
+	1    5200 3300
 	1    0    0    -1
 $EndComp
@@
 ACS_Relay_1
 $Comp
-L Relay Relay1
-U 1 1 59863DAD
-P 7000 1550
-F 0 "Relay1" H 7000 1550 60  0001 L BNN
-F 1 "Relay" H 7000 1550 60  0001 R TNN
-F 2 "Huellas de Componentes DqR:Relay" H 7000 1550 60  0001 C CNN
-F 3 "" H 7000 1550 60  0001 C CNN
-	1    7000 1550
-	1    0    0    -1
-$EndComp
-$Comp
-L Relay Relay2
-U 1 1 59863DC1
-P 7750 1550
-F 0 "Relay2" H 7750 1550 60  0001 L BNN
-F 1 "Relay" H 7750 1550 60  0001 R TNN
-F 2 "Huellas de Componentes DqR:Relay" H 7750 1550 60  0001 C CNN
-F 3 "" H 7750 1550 60  0001 C CNN
-	1    7750 1550
-	1    0    0    -1
-$EndComp
-NoConn ~ 7900 1800
-NoConn ~ 7550 1800
-$Comp
 L Screw_Terminal_1x04 J1
 U 1 1 59863F3A
-P 6100 1800
-F 0 "J1" H 6100 2250 50  0000 C TNN
-F 1 "Screw_Terminal_1x04" V 5950 1800 50  0000 C TNN
-F 2 "Connectors:bornier4" H 6100 1375 50  0001 C CNN
-F 3 "" H 6075 2000 50  0001 C CNN
-	1    6100 1800
+P 5900 850
+F 0 "J1" H 5900 1300 50  0000 C TNN
+F 1 "Screw_Terminal_1x04" V 5750 850 50  0000 C TNN
+F 2 "Connectors:bornier4" H 5900 425 50  0001 C CNN
+F 3 "" H 5875 1050 50  0001 C CNN
+	1    5900 850
 	0    -1   1    0
 $EndComp
@@
 L CONN_01X06 J2
 U 1 1 5987931C
-P 4500 3550
-F 0 "J2" H 4500 3900 50  0000 C CNN
-F 1 "CONN_01X06" V 4600 3550 50  0000 C CNN
-F 2 "Pin_Headers:Pin_Header_Straight_1x06_Pitch1.27mm" H 4500 3550 50  0001 C CNN
-F 3 "" H 4500 3550 50  0001 C CNN
-	1    4500 3550
+P 4150 4300
+F 0 "J2" H 4150 4650 50  0000 C CNN
+F 1 "CONN_01X06" V 4250 4300 50  0000 C CNN
+F 2 "Pin_Headers:Pin_Header_Straight_1x06_Pitch1.27mm" H 4150 4300 50  0001 C CNN
+F 3 "" H 4150 4300 50  0001 C CNN
+	1    4150 4300
 	0    -1   1    0
 $EndComp
-Wire Wire Line
-	6000 2100 6000 2000
-Connection ~ 5000 2300
-Wire Wire Line
-	5000 2300 5650 2300
-Connection ~ 5100 3050
-Wire Wire Line
-	5650 2500 5100 2500
-Wire Wire Line
-	5100 2500 5100 3800
-Connection ~ 4250 2800
-Wire Wire Line
-	4250 2900 4250 2800
-Wire Wire Line
-	4450 3350 4450 2400
-Wire Wire Line
-	4450 2400 5650 2400
-Wire Wire Line
-	4550 3350 4550 2950
-Wire Wire Line
-	4550 2950 5650 2950
-Wire Wire Line
-	7100 2600 7100 3050
-Wire Wire Line
-	7100 2600 8300 2600
-Wire Wire Line
-	8300 2600 8300 1800
-Wire Wire Line
-	4650 3350 4650 3250
-Wire Wire Line
-	4650 3250 6650 3250
-Wire Wire Line
-	6650 3250 6650 3550
-Wire Wire Line
-	6650 3550 8200 3550
-Wire Wire Line
-	8200 3550 8200 3000
-Wire Wire Line
-	5100 3050 5650 3050
-Wire Wire Line
-	4250 2800 4050 2800
-Wire Wire Line
-	4050 2800 4050 3800
-Wire Wire Line
-	4050 3800 8000 3800
-Connection ~ 7250 3800
-Wire Wire Line
-	7250 3800 7250 3000
-Wire Wire Line
-	8000 3800 8000 3000
-Connection ~ 4050 3350
-Connection ~ 5100 3800
-Wire Wire Line
-	4050 3350 4250 3350
-Wire Wire Line
-	4350 3350 4350 3300
-Wire Wire Line
-	4350 3300 4000 3300
-Wire Wire Line
-	4000 3300 4000 3850
-Wire Wire Line
-	4000 3850 8100 3850
-Wire Wire Line
-	5000 2300 5000 3850
-Connection ~ 5000 3850
-Wire Wire Line
-	8100 3850 8100 3000
-Connection ~ 7350 3850
-Wire Wire Line
-	7350 3000 7350 3850
-Wire Wire Line
-	4750 3350 6600 3350
-Wire Wire Line
-	6600 3350 6600 3600
-Wire Wire Line
-	6600 3600 7450 3600
-Wire Wire Line
-	7450 3600 7450 3000
-Connection ~ 5000 2850
-Connection ~ 6000 2100
-Connection ~ 7350 2100
-Wire Wire Line
-	8100 2100 8100 1800
-Wire Wire Line
-	4450 2100 8100 2100
-Wire Wire Line
-	7350 2100 7350 1800
-Wire Wire Line
-	4450 1750 4450 2100
-Wire Wire Line
-	5800 2000 5800 2050
-Wire Wire Line
-	5800 2050 4600 2050
-Wire Wire Line
-	4600 2050 4600 1750
 $Comp
-L PowerSupply_5V-RESCUE-Circuito_de_potencia_genérico PowerSupply_5V1
+L ACS712-20A ACS712-20A1
+U 1 1 59863649
+P 5200 2400
+F 0 "ACS712-20A1" V 5200 2400 60  0001 R TNN
+F 1 "ACS712-20A" H 5200 2400 60  0001 R TNN
+F 2 "Huellas de Componentes DqR:ACS712" H 5200 2400 60  0001 C CNN
+F 3 "" H 5200 2400 60  0001 C CNN
+	1    5200 2400
+	1    0    0    -1
+$EndComp
+$Comp
+L PowerSupply_5V PowerSupply_5V1
 U 1 1 598643CC
-P 4150 1650
-F 0 "PowerSupply_5V1" H 4150 1650 60  0001 L BNN
-F 1 "PowerSupply_5V" H 4150 1650 60  0001 R TNN
-F 2 "Huellas de Componentes DqR:PowerSupply5V" H 4150 1650 60  0001 C CNN
-F 3 "" H 4150 1650 60  0001 C CNN
-	1    4150 1650
+P 3350 1700
+F 0 "PowerSupply_5V1" H 3350 1700 60  0001 L BNN
+F 1 "PowerSupply_5V" H 3350 1700 60  0001 R TNN
+F 2 "Huellas de Componentes DqR:PowerSupply5V" H 3350 1700 60  0001 C CNN
+F 3 "" H 3350 1700 60  0001 C CNN
+	1    3350 1700
+	1    0    0    -1
+$EndComp
+$Comp
+L Relay Relay1
+U 1 1 59863DAD
+P 7300 1900
+F 0 "Relay1" H 7300 1900 60  0001 L BNN
+F 1 "Relay" H 7300 1900 60  0001 R TNN
+F 2 "Huellas de Componentes DqR:Relay" H 7300 1900 60  0001 C CNN
+F 3 "" H 7300 1900 60  0001 C CNN
+	1    7300 1900
 	1    0    0    -1
 $EndComp
 Wire Wire Line
-	4800 2850 5650 2850
+	9050 1500 9050 2150
 Wire Wire Line
-	4800 2900 4800 2850
+	5800 1500 5800 1050
+Connection ~ 7650 1500
+Wire Wire Line
+	7650 2150 7650 1500
+Wire Wire Line
+	3800 1300 3800 1800
+Connection ~ 5800 1500
+Wire Wire Line
+	3450 2950 3450 4650
+Wire Wire Line
+	3450 4100 3900 4100
+Wire Wire Line
+	4000 2950 4000 4100
+Wire Wire Line
+	3650 3450 5300 3450
+Connection ~ 4000 3450
+Wire Wire Line
+	5300 2550 4300 2550
+Wire Wire Line
+	4300 2550 4300 3450
+Connection ~ 4300 3450
+Wire Wire Line
+	5300 3650 3450 3650
+Connection ~ 3450 3650
+Wire Wire Line
+	5300 2750 4500 2750
+Wire Wire Line
+	4500 2750 4500 3650
+Connection ~ 4500 3650
+Wire Wire Line
+	5300 2650 4750 2650
+Wire Wire Line
+	4750 2650 4750 3800
+Wire Wire Line
+	4750 3800 4100 3800
+Wire Wire Line
+	4100 3800 4100 4100
+Wire Wire Line
+	5300 3550 4850 3550
+Wire Wire Line
+	4850 3550 4850 3900
+Wire Wire Line
+	4850 3900 4200 3900
+Wire Wire Line
+	4200 3900 4200 4100
+Wire Wire Line
+	7450 2150 7450 2750
+Wire Wire Line
+	7450 2750 6250 2750
+Wire Wire Line
+	6250 3650 7100 3650
+Wire Wire Line
+	7100 3650 7100 3000
+Wire Wire Line
+	7100 3000 9250 3000
+Wire Wire Line
+	9250 3000 9250 2150
+Wire Wire Line
+	6250 2550 6200 2550
+Wire Wire Line
+	6200 2550 6200 1050
+Wire Wire Line
+	6250 3450 6000 3450
+Wire Wire Line
+	6000 3450 6000 1050
+Wire Wire Line
+	8950 3400 8950 4650
+Wire Wire Line
+	8950 4650 3450 4650
+Connection ~ 3450 4100
+Wire Wire Line
+	7550 3400 7550 4650
+Connection ~ 7550 4650
+Wire Wire Line
+	9050 3400 9050 4850
+Wire Wire Line
+	9050 4850 3650 4850
+Wire Wire Line
+	3650 4850 3650 3450
+Wire Wire Line
+	7650 3400 7650 4850
+Connection ~ 7650 4850
 $Comp
-L ACS712-20A ACS712-20A1
-U 1 1 59863649
-P 5550 2150
-F 0 "ACS712-20A1" V 5550 2150 60  0001 R TNN
-F 1 "ACS712-20A" H 5550 2150 60  0001 R TNN
-F 2 "Huellas de Componentes DqR:ACS712" H 5550 2150 60  0001 C CNN
-F 3 "" H 5550 2150 60  0001 C CNN
-	1    5550 2150
+L Relay Relay2
+U 1 1 59863DC1
+P 8700 1900
+F 0 "Relay2" H 8700 1900 60  0001 L BNN
+F 1 "Relay" H 8700 1900 60  0001 R TNN
+F 2 "Huellas de Componentes DqR:Relay" H 8700 1900 60  0001 C CNN
+F 3 "" H 8700 1900 60  0001 C CNN
+	1    8700 1900
 	1    0    0    -1
 $EndComp
+NoConn ~ 8850 2150
+NoConn ~ 7850 2150
 Wire Wire Line
-	6400 2000 6400 2300
+	4500 1500 9050 1500
 Wire Wire Line
-	6400 2300 6600 2300
+	4500 1500 4500 2100
 Wire Wire Line
-	7150 1800 7150 2500
+	4500 2100 3650 2100
 Wire Wire Line
-	7150 2500 6600 2500
+	3650 2100 3650 1800
 Wire Wire Line
-	7100 3050 6600 3050
+	3800 1300 5600 1300
 Wire Wire Line
-	6200 2000 6200 2850
+	5600 1300 5600 1050
 Wire Wire Line
-	6200 2850 6600 2850
+	7750 3400 7750 4050
+Wire Wire Line
+	7750 4050 4400 4050
+Wire Wire Line
+	4400 4050 4400 4100
+Wire Wire Line
+	9150 3400 9150 3900
+Wire Wire Line
+	9150 3900 5250 3900
+Wire Wire Line
+	5250 3900 5250 4000
+Wire Wire Line
+	5250 4000 4300 4000
+Wire Wire Line
+	4300 4000 4300 4100
 $EndSCHEMATC
